File: pcb/fly2040_min/fly2040_min.kicad_pcb (KiCad board)
At the start: 4 copper layers, 19 x 15.6 mm, 39 parts, among them J1 Conn_01x01, J10 Conn_01x01, J2 Conn_01x01, J3 Conn_01x01, J4 Conn_01x01, J5 Conn_01x01, J6 Conn_01x01, J7 Conn_01x01, J8 Conn_01x06, J9 Conn_01x01, SW1 EVPAWED40, U1 RP2040, U2 W25Q16JVUXIQ, U5 XL-1010RGBC-WS2812B, X1 SMD-3225_4P_12.000MHZ_9PF

Commit message: Minor fixes to min board to prep for production run.
Parts:
- removed R8: 47, Resistor_SMD:R_0402_1005Metric
- added R3: 10k, Resistor_SMD:R_0402_1005Metric, F.Cu at (81.8, 60.6)
- moved U5 0.23 mm to (74.6, 63.5)
Connections:
- U1 pad 37: unconnected-(U1-GPIO25-Pad37) -> BOARD_DET
- U1 pad 38: Net-(U1-GPIO26_ADC0) -> NS_RST
Routing:
- net NS_RST: track 2.03 -> 5.35 mm
- net Net-(U1-GPIO26_ADC0): track 2.31 -> 0.00 mm
- net BOARD_DET: track 0.00 -> 1.88 mm
