File: pcb/fly2040_min/fly2040_min.kicad_sch (KiCad schematic)
At the start: 41 parts, among them J1 Conn_01x01, J10 Conn_01x01, J2 Conn_01x01, J3 Conn_01x01, J4 Conn_01x01, J5 Conn_01x01, J6 Conn_01x01, J7 Conn_01x01, J8 Conn_01x06, J9 Conn_01x01, SW1 EVPAWED40, U1 RP2040, U2 W25Q16JVUXIQ, U5 XL-1010RGBC-WS2812B, X1 SMD-3225_4P_12.000MHZ_9PF

Commit message: Minor fixes to min board to prep for production run.
Parts:
- removed R8: 47, R_0402_1005Metric, symbol jlcpcb-basic-resistor-0402:47
- added R3: 10k, R_0402_1005Metric, symbol jlcpcb-basic-resistor-0402:10k
Connections:
- net GND: now also R3.2
- net NS_RST: now also U1.38 (GPIO26_ADC0)
- net BOARD_DET: now reaches U1.37 (GPIO25)
- net BOARD_DET: now also R3.1
Changed lines of the file:
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@@
   (junction (at 138.43 44.45) (diameter 0) (color 0 0 0 0)
+  )
+  (junction (at 147.32 128.27) (diameter 0) (color 0 0 0 0)
   )
   (junction (at 106.68 46.99) (diameter 0) (color 0 0 0 0)
@@
     (stroke (width 0) (type default))
   )
-  (wire (pts (xy 127 133.35) (xy 125.73 133.35))
+  (wire (pts (xy 135.89 133.35) (xy 125.73 133.35))
     (stroke (width 0) (type default))
   )
@@
     (stroke (width 0) (type default))
   )
+  (wire (pts (xy 125.73 128.27) (xy 147.32 128.27))
+    (stroke (width 0) (type default))
+  )
   (wire (pts (xy 39.37 166.37) (xy 40.64 166.37))
     (stroke (width 0) (type default))
@@
     (stroke (width 0) (type default))
   )
-  (wire (pts (xy 135.89 133.35) (xy 132.08 133.35))
-    (stroke (width 0) (type default))
-  )
   (wire (pts (xy 135.89 140.97) (xy 132.08 140.97))
     (stroke (width 0) (type default))
@@
   )
   (wire (pts (xy 219.71 46.99) (xy 219.71 55.88))
+    (stroke (width 0) (type default))
+  )
+  (wire (pts (xy 149.86 128.27) (xy 147.32 128.27))
     (stroke (width 0) (type default))
   )
@@
     (property "Intersheetrefs" "${INTERSHEET_REFS}" (at 164.5847 110.49 0)
       (effects (font (size 1.27 1.27)) (justify right) hide)
+    )
+  )
+  (global_label "BOARD_DET" (shape input) (at 149.86 128.27 0) (fields_autoplaced)
+    (effects (font (size 1.27 1.27)) (justify left))
+    (property "Intersheetrefs" "${INTERSHEET_REFS}" (at 162.0472 128.27 0)
+      (effects (font (size 1.27 1.27)) (justify left) hide)
     )
   )
@@
     )
   )
+  (symbol (lib_id "power:GND") (at 147.32 133.35 0) (unit 1)
+    (in_bom yes) (on_board yes) (dnp no)
+    (property "Reference" "#PWR025" (at 147.32 139.7 0)
+      (effects (font (size 1.27 1.27)) hide)
+    )
+    (property "Value" "GND" (at 148.59 137.16 0)
+      (effects (font (size 1.27 1.27)))
+    )
+    (property "Footprint" "" (at 147.32 133.35 0)
+      (effects (font (size 1.27 1.27)) hide)
+    )
+    (property "Datasheet" "" (at 147.32 133.35 0)
+      (effects (font (size 1.27 1.27)) hide)
+    )
+    (pin "1")
+    (instances
+      (project "fly2040_min"
+        (path "/e63e39d7-6ac0-4ffd-8aa3-1841a4541b55"
+          (reference "#PWR025") (unit 1)
+        )
+      )
+    )
+  )
   (symbol (lib_id "power:+3V3") (at 102.87 38.1 0) (unit 1)
     (in_bom yes) (on_board yes) (dnp no)
@@
     )
   )
-  (symbol (lib_id "jlcpcb-basic-resistor-0402:47") (at 129.54 133.35 90) (unit 1)
-    (in_bom yes) (on_board yes) (dnp no)
-    (property "Reference" "R8" (at 133.35 132.08 90)
-      (effects (font (size 1.27 1.27)) hide)
-    )
-    (property "Value" "47" (at 129.54 133.35 90)
-      (effects (font (size 1.27 1.27)))
-    )
-    (property "Footprint" "R_0402_1005Metric" (at 129.54 133.35 0)
-      (effects (font (size 1.27 1.27)) hide)
-    )
-    (property "Datasheet" "https://datasheet.lcsc.com/lcsc/2110252230_UNI-ROYAL-Uniroyal-Elec-0402WGF470JTCE_C25118.pdf" (at 129.54 133.35 0)
-      (effects (font (size 1.27 1.27)) hide)
-    )
-    (property "LCSC" "C25118" (at 129.54 133.35 0)
-      (effects (font (size 0 0)) hide)
-    )
-    (property "MFG" "UNI-ROYAL(Uniroyal Elec)" (at 129.54 133.35 0)
-      (effects (font (size 0 0)) hide)
-    )
-    (property "MFGPN" "0402WGF470JTCE" (at 129.54 133.35 0)
-      (effects (font (size 0 0)) hide)
-    )
-    (pin "1")
-    (pin "2")
-    (instances
-      (project "fly2040_min"
-        (path "/e63e39d7-6ac0-4ffd-8aa3-1841a4541b55"
-          (reference "R8") (unit 1)
-        )
-      )
-    )
-  )
   (symbol (lib_id "power:GND") (at 148.59 93.98 0) (unit 1)
     (in_bom yes) (on_board yes) (dnp no)
@@
         )
       )
+    )
+  )
+  (symbol (lib_id "jlcpcb-basic-resistor-0402:10k") (at 147.32 130.81 0) (unit 1)
+    (in_bom yes) (on_board yes) (dnp no)
+    (property "Reference" "R3" (at 142.24 128.27 0)
+      (effects (font (size 1.27 1.27)) (justify left) hide)
+    )
+    (property "Value" "10k" (at 142.24 130.81 0)
+      (effects (font (size 1.27 1.27)) (justify left))
+    )
+    (property "Footprint" "R_0402_1005Metric" (at 147.32 130.81 0)
+      (effects (font (size 1.27 1.27)) hide)
+    )
+    (property "Datasheet" "https://datasheet.lcsc.com/lcsc/2110260030_UNI-ROYAL-Uniroyal-Elec-0402WGF1002TCE_C25744.pdf" (at 147.32 130.81 0)
+      (effects (font (size 1.27 1.27)) hide)
+    )
+    (property "LCSC" "C25744" (at 147.32 130.81 0)
+      (effects (font (size 0 0)) hide)
+    )
+    (property "MFG" "UNI-ROYAL(Uniroyal Elec)" (at 147.32 130.81 0)
+      (effects (font (size 0 0)) hide)
+    )
+    (property "MFGPN" "0402WGF1002TCE" (at 147.32 130.81 0)
+      (effects (font (size 0 0)) hide)
+    )
+    (pin "1")
+    (pin "2")
+    (instances
+      (project "fly2040_min"
+        (path "/e63e39d7-6ac0-4ffd-8aa3-1841a4541b55"
+          (reference "R3") (unit 1)
+        )
+      )
